File: kicad/LXKB.kicad_pcb (KiCad board)
At the start: 2 copper layers, 281.2 x 100.2 mm, 140 parts, among them J1 USB_C_Receptacle_USB2.0, SW1 SW_Push, SW10 SW_Push, SW11 SW_Push, SW12 SW_Push, SW13 SW_Push, SW14 SW_Push, SW15 SW_Push, SW16 SW_Push, SW17 SW_Push, SW18 SW_Push, SW19 SW_Push, SW2 SW_Push, SW20 SW_Push, SW21 SW_Push, SW22 SW_Push, SW23 SW_Push, SW24 SW_Push, SW25 SW_Push, SW26 SW_Push, SW27 SW_Push, SW28 SW_Push, SW29 SW_Push, SW3 SW_Push, SW30 SW_Push, SW31 SW_Push, SW32 SW_Push, SW33 SW_Push, SW34 SW_Push, SW35 SW_Push, SW36 SW_Push, SW37 SW_Push, SW38 SW_Push, SW39 SW_Push, SW4 SW_Push, SW40 SW_Push, SW41 SW_Push, SW42 SW_Push, SW43 SW_Push, SW44 SW_Push, SW45 SW_Push, SW46 SW_Push, SW47 SW_Push, SW48 SW_Push, SW49 SW_Push, SW5 SW_Push, SW50 SW_Push, SW51 SW_Push, SW52 SW_Push, SW53 SW_Push, SW54 SW_Push, SW55 SW_Push, SW56 SW_Push, SW57 SW_Push, SW58 SW_Push, SW59 SW_Push, SW6 SW_Push, SW60 SW_Push, SW7 SW_Push, SW8 SW_Push, SW9 SW_Push, U1 ATmega16U4-AU, U2 TPD2S017, Y1 Crystal_GND24

Commit message: Route PCB
Parts:
- removed ST42, ST53: MountingHole, Stabilizer_Cherry_MX_2u
- removed ST57: MountingHole, Stabilizer_Cherry_MX_6u
- moved J1 251.2 mm to (265.5, 19.9)
- moved U2 251.1 mm to (265.5, 27.9)
- moved C2 209.8 mm to (216.3, 100.5), turned to 270 degrees
- moved Y1 208.0 mm to (213.3, 100.6), turned to 90 degrees
- moved C1 206.4 mm to (213.3, 104.0), turned to 0 degrees
- moved R1 182.9 mm to (167.2, 93.3), turned to 0 degrees
- moved R2 182.5 mm to (167.2, 95.0), turned to 0 degrees
- moved RST 164.6 mm to (167.1, 100.6)
- moved R4 163.6 mm to (154.1, 103.5), turned to 270 degrees
- moved C4 155.4 mm to (141.5, 90.2)
- moved C8 155.4 mm to (141.5, 88.6)
- moved C7 153.4 mm to (136.0, 88.7)
- moved U1 150.0 mm to (133.1, 99.8), turned to 225 degrees
- moved C6 129.5 mm to (94.4, 95.8), turned to 270 degrees
- moved C3 125.9 mm to (94.4, 99.1), turned to 90 degrees
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Connections:
- U1 pad 7: (no net) -> VCC
Routing:
- net GND: track 0.00 -> 406.2 mm, vias 0 -> 5
- net VCC: track 69.3 -> 360.8 mm, vias 0 -> 4
- net COL14: track 0.00 -> 230.9 mm, vias 0 -> 3
- net u2/D-: track 4.46 -> 211.5 mm, vias 0 -> 2
- net u2/D+: track 4.47 -> 194.1 mm
- net ROW0: track 252.4 -> 421.5 mm, vias 0 -> 2
- net COL13: track 92.0 -> 244.0 mm, vias 0 -> 1
- net COL12: track 83.1 -> 212.8 mm, vias 0 -> 2
- net COL0: track 80.1 -> 192.7 mm
- net COL1: track 60.1 -> 170.8 mm
- net COL11: track 92.0 -> 193.2 mm
- net COL10: track 67.0 -> 161.5 mm, vias 0 -> 1
- net COL2: track 91.0 -> 182.8 mm, vias 0 -> 1
- net mcu/XTAL2: track 7.98 -> 88.2 mm, vias 0 -> 2
- net COL9: track 67.0 -> 145.1 mm, vias 0 -> 3
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Other:
- board size 281.2 x 100.2 mm -> 276.2 x 95.2 mm

Commit message: Add rounding to edgecut of PCB
Parts:
- moved R4 12.5 mm to (165.6, 108.4), turned to 0 degrees
Routing:
- net mcu/~RESET: track 41.3 -> 60.6 mm, vias 2 -> 4
- net ROW4: track 259.6 -> 263.9 mm
- net COL0: track 192.7 -> 196.9 mm
- net VCC: track 360.8 -> 357.0 mm, vias 4 -> 5
- net ROW0: track 421.5 -> 422.9 mm
- net mcu/D-: track 36.0 -> 37.1 mm
- net GND: track 406.2 -> 407.2 mm
- net mcu/D+: track 35.9 -> 36.7 mm
- net COL11: track 193.2 -> 193.8 mm
- net mcu/UCAP: track 10.7 -> 11.4 mm
- net COL12: track 212.8 -> 213.4 mm
- net COL6: track 102.1 -> 102.6 mm
- net COL2: track 182.8 -> 183.3 mm
- net COL10: track 161.5 -> 162.1 mm
- net ROW2: track 277.1 -> 277.7 mm
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Other:
- outline, holes or cut-outs redrawn
- board text added: "LXKB v1"
